Commit message: initial orientation, initial rotation, initial approach added

File: OpenSai/cs225a/urdf_models/panda/panda_arm_hand.urdf (robot description, URDF)
Before this commit: robot panda_arm_hand, 10 links, 9 joints
Links:
- removed link leftfinger
- removed link rightfinger
- added link sponge, mass 0.1; collision cylinder length=0.03 radius=0.05; visual cylinder length=0.03 radius=0.05
- link link7: geometry visual mesh filename=meshes/visual/link7.obj
Joints:
- removed joint finger_joint1
- removed joint finger_joint2
- added joint sponge: type fixed, parent link7, child sponge, origin xyz=0 0 0 rpy=0 0 0
